File: dribbler_driver_ver.4/dribbler_driver.kicad_sch (KiCad schematic)
At the start: 101 parts, among them J1 Conn_01x04_Pin, J3 Conn_01x02_MountingPin, J4 Conn_01x02_MountingPin, J5 Conn_01x02_Pin, J6 Conn_01x08_Socket, Q1 WSD4070DN, Q10 WSD4070DN, Q2 WSD4070DN, Q5 WSD4070DN, Q6 WSD4070DN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

Commit message: updated RY8411 footprint
Parts:
- RY8411: footprint Package_DFN_QFN:DFN-8-1EP_3x3mm_P0.65mm_EP1.5x2.25mm -> Package_TO_SOT_SMD:SOT-23-6_Handsoldering
Changed lines of the file:
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@@
 			)
 		)
-		(property "Footprint" "Package_DFN_QFN:DFN-8-1EP_3x3mm_P0.65mm_EP1.5x2.25mm"
+		(property "Footprint" "Package_TO_SOT_SMD:SOT-23-6_Handsoldering"
 			(at 208.28 30.48 0)
 			(effects
