File: dribbler_driver_ver.5.3/dribbler_driver.kicad_pcb (KiCad board)
At the start: 4 copper layers, 77.6 x 32.1 mm, 97 parts, among them J1 Conn_01x04_Pin, J3 Conn_01x02_MountingPin, J4 Conn_01x02_MountingPin, J5 Conn_01x02_Pin, J6 Conn_01x08_Socket, Q1 WSD4070DN, Q10 WSD4070DN, Q2 WSD4070DN, Q5 WSD4070DN, Q6 WSD4070DN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

Commit message: clean up
Parts:
- removed C3: 0.01u, Capacitor_SMD:C_0603_1608Metric_Pad1.08x0.95mm_HandSolder
- added G***: LOGO, LOGO, B.Cu at (79.4, 34.0)
- moved J5 26.5 mm to (88.3, 37.5)
- moved USART1 26.0 mm to (88.2, 29.3)
- moved C2 25.7 mm to (65.5, 39.7)
- moved D1 25.7 mm to (75.5, 36.8)
- moved D8 25.7 mm to (65.5, 41.5)
- moved R19 25.7 mm to (69.7, 25.2)
- moved C1 25.7 mm to (77.2, 40.4)
- moved C10 25.7 mm to (70.3, 28.0)
- moved C12 25.7 mm to (57.7, 32.0)
- moved C14 25.7 mm to (59.2, 21.7)
- moved C15 25.7 mm to (28.8, 25.0)
- moved C20 25.7 mm to (39.1, 44.1)
- moved C21 25.7 mm to (57.2, 37.3)
- moved C23 25.7 mm to (39.9, 34.4)
- moved C28 25.7 mm to (62.7, 37.4)
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Routing:
- net USART2_TX: track 24.5 -> 25.0 mm
Other:
- board size 77.6 x 32.1 mm -> 77.7 x 32.1 mm
- board text added: "Dribbler 24V 60W BLDC FOC Driver Gen1"
- board text added: "JLCJLCJLCJLCJLCCJLC"
- board text added: "Steven. Z. Jonas. Z."
