File: dribbler_driver_ver.5.3/dribbler_driver.kicad_sch (KiCad schematic)
At the start: 97 parts, among them J1 Conn_01x04_Pin, J3 Conn_01x02_MountingPin, J4 Conn_01x02_MountingPin, J5 Conn_01x02_Pin, J6 Conn_01x08_Socket, Q1 WSD4070DN, Q10 WSD4070DN, Q2 WSD4070DN, Q5 WSD4070DN, Q6 WSD4070DN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

Commit message: clean up
Other:
- moved on the sheet: C1, C10, C11, C12, C13, C14, C15, C16, C17, C18, C2, C20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
