File: dribbler_driver_ver.6/dribbler_driver.kicad_sch (KiCad schematic)
At the start: 99 parts, among them J1 Conn_01x04_MountingPin, J2 Conn_01x03_MountingPin, J3 Conn_01x02_MountingPin, J4 Conn_01x02_MountingPin, J5 Conn_01x02_Pin, J6 Conn_01x08_MountingPin, J7 Conn_01x02_MountingPin, J8 Conn_01x03_MountingPin, Q1 WSD4070DN, Q10 WSD4070DN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

Commit message: gen 6 production
Parts:
- added R? (x2): 0.05, Resistor_SMD:R_1206_3216Metric, symbol Device:R
- C2: renamed from C4; value 0.01u -> 2n
- C3, C5: value 0.01u -> 2n
Changed lines of the file:
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@@
 			)
 		)
-		(property "Value" "0.01u"
+		(property "Value" "2n"
 			(at 321.056 121.666 0)
 			(effects
@@
 		(on_board yes)
 		(dnp no)
-		(property "Reference" "C4"
+		(property "Reference" "C2"
 			(at 309.372 117.094 0)
 			(effects
@@
 			)
 		)
-		(property "Value" "0.01u"
+		(property "Value" "2n"
 			(at 309.372 121.666 0)
 			(effects
@@
 			(project "dribbler_driver"
 				(path "/16386afa-d57f-4224-8aa0-968af24bcdeb"
-					(reference "C4")
+					(reference "C2")
 					(unit 1)
 				)
@@
 			)
 		)
-		(property "Value" "0.01u"
+		(property "Value" "2n"
 			(at 298.196 121.92 0)
 			(effects
@@
 	)
 	(symbol
+		(lib_id "Device:R")
+		(at 27.94 87.63 180)
+		(unit 1)
+		(exclude_from_sim no)
+		(in_bom yes)
+		(on_board yes)
+		(dnp no)
+		(property "Reference" "R?"
+			(at 25.908 85.852 90)
+			(effects
+				(font
+					(size 1.27 1.27)
+				)
+				(justify left)
+			)
+		)
+		(property "Value" "0.05"
+			(at 23.622 84.328 90)
+			(effects
+				(font
+					(size 1.27 1.27)
+				)
+				(justify left)
+			)
+		)
+		(property "Footprint" "Resistor_SMD:R_1206_3216Metric"
+			(at 29.718 87.63 90)
+			(effects
+				(font
+					(size 1.27 1.27)
+				)
+				(hide yes)
+			)
+		)
+		(property "Datasheet" "~"
+			(at 27.94 87.63 0)
+			(effects
+				(font
+					(size 1.27 1.27)
+				)
+				(hide yes)
+			)
+		)
+		(property "Description" ""
+			(at 27.94 87.63 0)
+			(effects
+				(font
+					(size 1.27 1.27)
+				)
+				(hide yes)
+			)
+		)
+		(pin "1"
+		)
+		(pin "2"
+		)
+		(instances
+			(project "dribbler_driver"
+				(path "/16386afa-d57f-4224-8aa0-968af24bcdeb"
+					(reference "R?")
+					(unit 1)
+				)
+			)
+		)
+	)
+	(symbol
 		(lib_id "Connector:Conn_01x02_Pin")
 		(at 374.65 116.84 180)
@@
 					(unit 1)
 				)
+			)
+		)
+	)
+	(symbol
+		(lib_id "Device:R")
+		(at 30.48 116.84 180)
+		(unit 1)
+		(exclude_from_sim no)
+		(in_bom yes)
+		(on_board yes)
+		(dnp no)
+		(property "Reference" "R?"
+			(at 28.448 115.062 90)
+			(effects
+				(font
+					(size 1.27 1.27)
+				)
+				(justify left)
+			)
+		)
+		(property "Value" "0.05"
+			(at 26.162 113.538 90)
+			(effects
+				(font
+					(size 1.27 1.27)
+				)
+				(justify left)
+			)
+		)
+		(property "Footprint" "Resistor_SMD:R_1206_3216Metric"
+			(at 32.258 116.84 90)
+			(effects
+				(font
+					(size 1.27 1.27)
+				)
+				(hide yes)
+			)
+		)
+		(property "Datasheet" "~"
+			(at 30.48 116.84 0)
+			(effects
+				(font
+					(size 1.27 1.27)
+				)
+				(hide yes)
+			)
+		)
+		(property "Description" ""
+			(at 30.48 116.84 0)
+			(effects
+				(font
+					(size 1.27 1.27)
+				)
+				(hide yes)
+			)
+		)
+		(pin "1"
+		)
+		(pin "2"
+		)
+		(instances
+			(project "dribbler_driver"
+				(path "/16386afa-d57f-4224-8aa0-968af24bcdeb"
+					(reference "R?")
+					(unit 1)
+				)
